File: parts/extruder pcb/extruderevolved.kicad_pcb (KiCad board)
At the start: 2 copper layers, 68 x 57 mm, 8 parts, among them CN1 B-3102R24P-A000, CN2 HC-1.25-2PWT, CN3 HC-1.25-3PWT, CN4 HC-1.25-4PWT, CN5 HC-1.25-5PWT, CN6 X2011WRS-02A-9TSN, CN7 HC-1.25-2PWT, CN8 HC-1.25-2PWT

Commit message: Add files via upload
Parts:
- moved CN2 1.00 mm to (182.0, 112.0)
- moved CN5 0.88 mm to (171.1, 112.0)
Routing:
- net GND: track 0.00 -> 129.4 mm
- net Part Cooling Fan+: track 0.00 -> 68.7 mm
- net Part Cooling Fan-: track 0.00 -> 60.2 mm
- net Probe #2: track 0.00 -> 59.6 mm, vias 0 -> 1
- net Probe #4: track 0.00 -> 57.7 mm, vias 0 -> 1
- net Termistor-: track 0.00 -> 56.6 mm, vias 0 -> 1
- net Heater-: track 0.00 -> 56.6 mm, vias 0 -> 1
- net Thermistor+: track 0.00 -> 53.6 mm, vias 0 -> 1
- net E Motor #4: track 0.00 -> 51.1 mm
- net Probe #5: track 0.00 -> 50.2 mm, vias 0 -> 1
- net Heater+: track 0.00 -> 50.2 mm
- net Probe #3: track 0.00 -> 50.0 mm, vias 0 -> 1
- net Probe #1: track 0.00 -> 49.8 mm, vias 0 -> 1
- net E Motor #3: track 0.00 -> 43.8 mm
- net E Motor #2: track 0.00 -> 43.7 mm
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Other:
- outline, holes or cut-outs redrawn
